File: BasicCom.sch (KiCad schematic (older format))
At the start: 9 parts, among them P10 UART_2, P11 I2C, P9 UART_1

Commit message: Adding Hermes 2 schematic files.
Parts:
- P3: renamed from P9; value UART_1 -> UART_0; footprint Footprints:Conn_01x03 -> (none); symbol CONN_01X03 -> Conn_01x03
- P4: renamed from P10; value UART_2 -> UART_1; footprint Footprints:Conn_01x03 -> (none); symbol CONN_01X03 -> Conn_01x03
- P5: renamed from P11; footprint Footprints:Conn_01x03 -> (none); symbol CONN_01X03 -> Conn_01x03
- R10: renamed from R22; footprint Footprints:R_CMS1206 -> (none)
- R11: renamed from R23; footprint Footprints:R_CMS1206 -> (none)
- R6: renamed from R18; footprint Footprints:R_CMS1206 -> (none)
- R7: renamed from R19; footprint Footprints:R_CMS1206 -> (none)
- R8: renamed from R20; footprint Footprints:R_CMS1206 -> (none)
- R9: renamed from R21; footprint Footprints:R_CMS1206 -> (none)
Connections:
- net labels added: +3.3V, RX0, TX0
- net labels removed: +5V, RX2, TX2
Changed lines of the file:
@@
 EESchema Schematic File Version 2
-LIBS:power
 LIBS:device
-LIBS:transistors
 LIBS:conn
-LIBS:linear
-LIBS:regul
-LIBS:74xx
-LIBS:cmos4000
-LIBS:adc-dac
-LIBS:memory
-LIBS:xilinx
-LIBS:microcontrollers
-LIBS:dsp
-LIBS:microchip
-LIBS:analog_switches
-LIBS:motorola
-LIBS:texas
-LIBS:intel
-LIBS:audio
-LIBS:interface
-LIBS:digital-audio
-LIBS:philips
-LIBS:display
-LIBS:cypress
-LIBS:siliconi
-LIBS:opto
-LIBS:atmel
-LIBS:contrib
-LIBS:valves
-LIBS:Hermes-cache
 EELAYER 25 0
 EELAYER END
 $Descr A4 11693 8268
 encoding utf-8
-Sheet 9 17
-Title ""
+Sheet 3 18
+Title "Hermes2 basic communication buses"
 Date ""
-Rev ""
+Rev "rev1"
 Comp ""
-Comment1 ""
+Comment1 "With 3.3V pull-ups"
 Comment2 ""
 Comment3 ""
@@
 $EndDescr
 $Comp
-L CONN_01X03 P9
+L Conn_01x03 P3
 U 1 1 55E8DDC2
 P 6450 3500
-F 0 "P9" H 6450 3700 50  0000 C CNN
-F 1 "UART_1" V 6550 3500 50  0000 C CNN
-F 2 "Footprints:Conn_01x03" H 6450 3500 60  0001 C CNN
+F 0 "P3" H 6450 3700 50  0000 C CNN
+F 1 "UART_0" V 6550 3500 50  0000 C CNN
+F 2 "" H 6450 3500 60  0001 C CNN
 F 3 "" H 6450 3500 60  0000 C CNN
 	1    6450 3500
@@
 $EndComp
 $Comp
-L CONN_01X03 P10
+L Conn_01x03 P4
 U 1 1 55E8DDF7
 P 6450 4050
-F 0 "P10" H 6450 4250 50  0000 C CNN
-F 1 "UART_2" V 6550 4050 50  0000 C CNN
-F 2 "Footprints:Conn_01x03" H 6450 4050 60  0001 C CNN
+F 0 "P4" H 6450 4250 50  0000 C CNN
+F 1 "UART_1" V 6550 4050 50  0000 C CNN
+F 2 "" H 6450 4050 60  0001 C CNN
 F 3 "" H 6450 4050 60  0000 C CNN
 	1    6450 4050
@@
 $EndComp
 $Comp
-L CONN_01X03 P11
+L Conn_01x03 P5
 U 1 1 55E8DE74
 P 6450 4600
-F 0 "P11" H 6450 4800 50  0000 C CNN
+F 0 "P5" H 6450 4800 50  0000 C CNN
 F 1 "I2C" V 6550 4600 50  0000 C CNN
-F 2 "Footprints:Conn_01x03" H 6450 4600 60  0001 C CNN
+F 2 "" H 6450 4600 60  0001 C CNN
 F 3 "" H 6450 4600 60  0000 C CNN
 	1    6450 4600
@@
 GND
 Text HLabel 5150 3400 0    60   Input ~ 0
+TX0
+Text HLabel 5150 3600 0    60   Output ~ 0
+RX0
+Text HLabel 5150 3950 0    60   Input ~ 0
 TX1
-Text HLabel 5150 3600 0    60   Output ~ 0
+Text HLabel 5150 4150 0    60   Output ~ 0
 RX1
-Text HLabel 5150 3950 0    60   Input ~ 0
-TX2
-Text HLabel 5150 4150 0    60   Output ~ 0
-RX2
 Text HLabel 5150 4500 0    60   Input ~ 0
 SCL
@@
 SDA
 Text HLabel 5150 2550 0    60   Input ~ 0
-+5V
++3.3V
 $Comp
-L R R18
+L R R6
 U 1 1 5602B2EE
 P 5200 2800
-F 0 "R18" V 5280 2800 50  0000 C CNN
+F 0 "R6" V 5280 2800 50  0000 C CNN
 F 1 "10kΩ" V 5200 2800 50  0000 C CNN
-F 2 "Footprints:R_CMS1206" V 5130 2800 30  0001 C CNN
+F 2 "" V 5130 2800 30  0001 C CNN
 F 3 "" H 5200 2800 30  0000 C CNN
 	1    5200 2800
@@
 	5150 3500 6250 3500
 $Comp
-L R R19
+L R R7
 U 1 1 5602B4FB
 P 5400 2800
-F 0 "R19" V 5480 2800 50  0000 C CNN
+F 0 "R7" V 5480 2800 50  0000 C CNN
 F 1 "10kΩ" V 5400 2800 50  0000 C CNN
-F 2 "Footprints:R_CMS1206" V 5330 2800 30  0001 C CNN
+F 2 "" V 5330 2800 30  0001 C CNN
 F 3 "" H 5400 2800 30  0000 C CNN
 	1    5400 2800
@@
 	5150 3950 6250 3950
 $Comp
-L R R20
+L R R8
 U 1 1 5602B666
 P 5600 2800
-F 0 "R20" V 5680 2800 50  0000 C CNN
+F 0 "R8" V 5680 2800 50  0000 C CNN
 F 1 "10kΩ" V 5600 2800 50  0000 C CNN
-F 2 "Footprints:R_CMS1206" V 5530 2800 30  0001 C CNN
+F 2 "" V 5530 2800 30  0001 C CNN
 F 3 "" H 5600 2800 30  0000 C CNN
 	1    5600 2800
@@
 $EndComp
 $Comp
-L R R21
+L R R9
 U 1 1 5602B66C
 P 5800 2800
-F 0 "R21" V 5880 2800 50  0000 C CNN
+F 0 "R9" V 5880 2800 50  0000 C CNN
 F 1 "10kΩ" V 5800 2800 50  0000 C CNN
-F 2 "Footprints:R_CMS1206" V 5730 2800 30  0001 C CNN
+F 2 "" V 5730 2800 30  0001 C CNN
 F 3 "" H 5800 2800 30  0000 C CNN
 	1    5800 2800
@@
 	6250 4700 5150 4700
 $Comp
-L R R22
+L R R10
 U 1 1 5602BC08
 P 6000 2800
-F 0 "R22" V 6080 2800 50  0000 C CNN
+F 0 "R10" V 6080 2800 50  0000 C CNN
 F 1 "10kΩ" V 6000 2800 50  0000 C CNN
-F 2 "Footprints:R_CMS1206" V 5930 2800 30  0001 C CNN
+F 2 "" V 5930 2800 30  0001 C CNN
 F 3 "" H 6000 2800 30  0000 C CNN
 	1    6000 2800
@@
 $EndComp
 $Comp
-L R R23
+L R R11
 U 1 1 5602BC0E
 P 6200 2800
-F 0 "R23" V 6280 2800 50  0000 C CNN
+F 0 "R11" V 6280 2800 50  0000 C CNN
 F 1 "10kΩ" V 6200 2800 50  0000 C CNN
-F 2 "Footprints:R_CMS1206" V 6130 2800 30  0001 C CNN
+F 2 "" V 6130 2800 30  0001 C CNN
 F 3 "" H 6200 2800 30  0000 C CNN
 	1    6200 2800

Commit message: Changing I2C pull-up resistors to 2kohm to allow I2C bus to work in fast-mode.
Parts:
- R10, R11: value 10kΩ -> 2kΩ
Changed lines of the file:
@@
 P 6000 2800
 F 0 "R10" V 6080 2800 50  0000 C CNN
-F 1 "10kΩ" V 6000 2800 50  0000 C CNN
+F 1 "2kΩ" V 6000 2800 50  0000 C CNN
 F 2 "" V 5930 2800 30  0001 C CNN
 F 3 "" H 6000 2800 30  0000 C CNN
@@
 P 6200 2800
 F 0 "R11" V 6280 2800 50  0000 C CNN
-F 1 "10kΩ" V 6200 2800 50  0000 C CNN
+F 1 "2kΩ" V 6200 2800 50  0000 C CNN
 F 2 "" V 6130 2800 30  0001 C CNN
 F 3 "" H 6200 2800 30  0000 C CNN

Commit message: Changing some value fields on the schematics for a better grouped_csv BOM generation.
Parts:
- P3: value UART_0 -> UART_IO
- P4: value UART_1 -> UART_IO
- P5: value I2C -> I2C_IO
Changed lines of the file:
@@
 P 6450 3500
 F 0 "P3" H 6450 3700 50  0000 C CNN
-F 1 "UART_0" V 6550 3500 50  0000 C CNN
+F 1 "UART_IO" V 6550 3500 50  0000 C CNN
 F 2 "" H 6450 3500 60  0001 C CNN
 F 3 "" H 6450 3500 60  0000 C CNN
@@
 P 6450 4050
 F 0 "P4" H 6450 4250 50  0000 C CNN
-F 1 "UART_1" V 6550 4050 50  0000 C CNN
+F 1 "UART_IO" V 6550 4050 50  0000 C CNN
 F 2 "" H 6450 4050 60  0001 C CNN
 F 3 "" H 6450 4050 60  0000 C CNN
@@
 P 6450 4600
 F 0 "P5" H 6450 4800 50  0000 C CNN
-F 1 "I2C" V 6550 4600 50  0000 C CNN
+F 1 "I2C_IO" V 6550 4600 50  0000 C CNN
 F 2 "" H 6450 4600 60  0001 C CNN
 F 3 "" H 6450 4600 60  0000 C CNN

Commit message: Updating the schematic's annotations.
Parts:
- renumbered P3 to P301, P4 to P302, P5 to P303, R6 to R301, R7 to R302, R8 to R303, R9 to R304, R10 to R305, R11 to R306
Changed lines of the file:
@@
 $EndDescr
 $Comp
-L Conn_01x03 P3
+L Conn_01x03 P301
 U 1 1 55E8DDC2
 P 6450 3500
-F 0 "P3" H 6450 3700 50  0000 C CNN
+F 0 "P301" H 6450 3700 50  0000 C CNN
 F 1 "UART_IO" V 6550 3500 50  0000 C CNN
 F 2 "" H 6450 3500 60  0001 C CNN
@@
 $EndComp
 $Comp
-L Conn_01x03 P4
+L Conn_01x03 P302
 U 1 1 55E8DDF7
 P 6450 4050
-F 0 "P4" H 6450 4250 50  0000 C CNN
+F 0 "P302" H 6450 4250 50  0000 C CNN
 F 1 "UART_IO" V 6550 4050 50  0000 C CNN
 F 2 "" H 6450 4050 60  0001 C CNN
@@
 $EndComp
 $Comp
-L Conn_01x03 P5
+L Conn_01x03 P303
 U 1 1 55E8DE74
 P 6450 4600
-F 0 "P5" H 6450 4800 50  0000 C CNN
+F 0 "P303" H 6450 4800 50  0000 C CNN
 F 1 "I2C_IO" V 6550 4600 50  0000 C CNN
 F 2 "" H 6450 4600 60  0001 C CNN
@@
 +3.3V
 $Comp
-L R R6
+L R R301
 U 1 1 5602B2EE
 P 5200 2800
-F 0 "R6" V 5280 2800 50  0000 C CNN
+F 0 "R301" V 5280 2800 50  0000 C CNN
 F 1 "10kΩ" V 5200 2800 50  0000 C CNN
 F 2 "" V 5130 2800 30  0001 C CNN
@@
 	5150 3500 6250 3500
 $Comp
-L R R7
+L R R302
 U 1 1 5602B4FB
 P 5400 2800
-F 0 "R7" V 5480 2800 50  0000 C CNN
+F 0 "R302" V 5480 2800 50  0000 C CNN
 F 1 "10kΩ" V 5400 2800 50  0000 C CNN
 F 2 "" V 5330 2800 30  0001 C CNN
@@
 	5150 3950 6250 3950
 $Comp
-L R R8
+L R R303
 U 1 1 5602B666
 P 5600 2800
-F 0 "R8" V 5680 2800 50  0000 C CNN
+F 0 "R303" V 5680 2800 50  0000 C CNN
 F 1 "10kΩ" V 5600 2800 50  0000 C CNN
 F 2 "" V 5530 2800 30  0001 C CNN
@@
 $EndComp
 $Comp
-L R R9
+L R R304
 U 1 1 5602B66C
 P 5800 2800
-F 0 "R9" V 5880 2800 50  0000 C CNN
+F 0 "R304" V 5880 2800 50  0000 C CNN
 F 1 "10kΩ" V 5800 2800 50  0000 C CNN
 F 2 "" V 5730 2800 30  0001 C CNN
@@
 	6250 4700 5150 4700
 $Comp
-L R R10
+L R R305
 U 1 1 5602BC08
 P 6000 2800
-F 0 "R10" V 6080 2800 50  0000 C CNN
+F 0 "R305" V 6080 2800 50  0000 C CNN
 F 1 "2kΩ" V 6000 2800 50  0000 C CNN
 F 2 "" V 5930 2800 30  0001 C CNN
@@
 $EndComp
 $Comp
-L R R11
+L R R306
 U 1 1 5602BC0E
 P 6200 2800
-F 0 "R11" V 6280 2800 50  0000 C CNN
+F 0 "R306" V 6280 2800 50  0000 C CNN
 F 1 "2kΩ" V 6200 2800 50  0000 C CNN
 F 2 "" V 6130 2800 30  0001 C CNN

Commit message: Setting the schematic's footprints.
Parts:
- P301, P302, P303: footprint (none) -> Connectors_Molex:Molex_KK-6410-03_03x2.54mm_Straight
- R301, R302, R303, R304, R305, R306: footprint (none) -> Resistors_SMD:R_1206_HandSoldering
Changed lines of the file:
@@
 F 0 "P301" H 6450 3700 50  0000 C CNN
 F 1 "UART_IO" V 6550 3500 50  0000 C CNN
-F 2 "" H 6450 3500 60  0001 C CNN
+F 2 "Connectors_Molex:Molex_KK-6410-03_03x2.54mm_Straight" H 6450 3500 60  0001 C CNN
 F 3 "" H 6450 3500 60  0000 C CNN
 	1    6450 3500
@@
 F 0 "P302" H 6450 4250 50  0000 C CNN
 F 1 "UART_IO" V 6550 4050 50  0000 C CNN
-F 2 "" H 6450 4050 60  0001 C CNN
+F 2 "Connectors_Molex:Molex_KK-6410-03_03x2.54mm_Straight" H 6450 4050 60  0001 C CNN
 F 3 "" H 6450 4050 60  0000 C CNN
 	1    6450 4050
@@
 F 0 "P303" H 6450 4800 50  0000 C CNN
 F 1 "I2C_IO" V 6550 4600 50  0000 C CNN
-F 2 "" H 6450 4600 60  0001 C CNN
+F 2 "Connectors_Molex:Molex_KK-6410-03_03x2.54mm_Straight" H 6450 4600 60  0001 C CNN
 F 3 "" H 6450 4600 60  0000 C CNN
 	1    6450 4600
@@
 F 0 "R301" V 5280 2800 50  0000 C CNN
 F 1 "10kΩ" V 5200 2800 50  0000 C CNN
-F 2 "" V 5130 2800 30  0001 C CNN
+F 2 "Resistors_SMD:R_1206_HandSoldering" V 5130 2800 30  0001 C CNN
 F 3 "" H 5200 2800 30  0000 C CNN
 	1    5200 2800
@@
 F 0 "R302" V 5480 2800 50  0000 C CNN
 F 1 "10kΩ" V 5400 2800 50  0000 C CNN
-F 2 "" V 5330 2800 30  0001 C CNN
+F 2 "Resistors_SMD:R_1206_HandSoldering" V 5330 2800 30  0001 C CNN
 F 3 "" H 5400 2800 30  0000 C CNN
 	1    5400 2800
@@
 F 0 "R303" V 5680 2800 50  0000 C CNN
 F 1 "10kΩ" V 5600 2800 50  0000 C CNN
-F 2 "" V 5530 2800 30  0001 C CNN
+F 2 "Resistors_SMD:R_1206_HandSoldering" V 5530 2800 30  0001 C CNN
 F 3 "" H 5600 2800 30  0000 C CNN
 	1    5600 2800
@@
 F 0 "R304" V 5880 2800 50  0000 C CNN
 F 1 "10kΩ" V 5800 2800 50  0000 C CNN
-F 2 "" V 5730 2800 30  0001 C CNN
+F 2 "Resistors_SMD:R_1206_HandSoldering" V 5730 2800 30  0001 C CNN
 F 3 "" H 5800 2800 30  0000 C CNN
 	1    5800 2800
@@
 F 0 "R305" V 6080 2800 50  0000 C CNN
 F 1 "2kΩ" V 6000 2800 50  0000 C CNN
-F 2 "" V 5930 2800 30  0001 C CNN
+F 2 "Resistors_SMD:R_1206_HandSoldering" V 5930 2800 30  0001 C CNN
 F 3 "" H 6000 2800 30  0000 C CNN
 	1    6000 2800
@@
 F 0 "R306" V 6280 2800 50  0000 C CNN
 F 1 "2kΩ" V 6200 2800 50  0000 C CNN
-F 2 "" V 6130 2800 30  0001 C CNN
+F 2 "Resistors_SMD:R_1206_HandSoldering" V 6130 2800 30  0001 C CNN
 F 3 "" H 6200 2800 30  0000 C CNN
 	1    6200 2800
