File: CANCom.sch (KiCad schematic (older format))
At the start: 4 parts, among them J1 Conn_01x03, J2 Conn_01x03, U3 SN65HVD232

Commit message: Changing some value fields on the schematics for a better grouped_csv BOM generation.
Parts:
- P19: renamed from J1; value Conn_01x03 -> CAN_IO
- P20: renamed from J2; value Conn_01x03 -> CAN_IO
Changed lines of the file:
@@
 TX
 $Comp
-L Conn_01x03 J1
+L Conn_01x03 P19
 U 1 1 5A003923
 P 6350 3650
-F 0 "J1" H 6350 3850 50  0000 C CNN
-F 1 "Conn_01x03" H 6350 3450 50  0000 C CNN
+F 0 "P19" H 6350 3850 50  0000 C CNN
+F 1 "CAN_IO" H 6350 3450 50  0000 C CNN
 F 2 "" H 6350 3650 50  0001 C CNN
 F 3 "" H 6350 3650 50  0001 C CNN
@@
 $EndComp
 $Comp
-L Conn_01x03 J2
+L Conn_01x03 P20
 U 1 1 5A00395B
 P 6850 3650
-F 0 "J2" H 6850 3850 50  0000 C CNN
-F 1 "Conn_01x03" H 6850 3450 50  0000 C CNN
+F 0 "P20" H 6850 3850 50  0000 C CNN
+F 1 "CAN_IO" H 6850 3450 50  0000 C CNN
 F 2 "" H 6850 3650 50  0001 C CNN
 F 3 "" H 6850 3650 50  0001 C CNN

Commit message: Updating the schematic's annotations.
Parts:
- renumbered C5 to C401, P19 to P401, P20 to P402, U3 to U401
Changed lines of the file:
@@
 $EndDescr
 $Comp
-L SN65HVD232 U3
+L SN65HVD232 U401
 U 1 1 5A003547
 P 5650 3950
-F 0 "U3" H 5550 4350 50  0000 R CNN
+F 0 "U401" H 5550 4350 50  0000 R CNN
 F 1 "SN65HVD232" H 5550 4250 50  0000 R CNN
 F 2 "" H 5650 3450 50  0001 C CNN
@@
 GND
 $Comp
-L C C5
+L C C401
 U 1 1 5A003774
 P 4800 4300
-F 0 "C5" H 4825 4400 50  0000 L CNN
+F 0 "C401" H 4825 4400 50  0000 L CNN
 F 1 "100nF" H 4825 4200 50  0000 L CNN
 F 2 "" H 4838 4150 50  0001 C CNN
@@
 TX
 $Comp
-L Conn_01x03 P19
+L Conn_01x03 P401
 U 1 1 5A003923
 P 6350 3650
-F 0 "P19" H 6350 3850 50  0000 C CNN
+F 0 "P401" H 6350 3850 50  0000 C CNN
 F 1 "CAN_IO" H 6350 3450 50  0000 C CNN
 F 2 "" H 6350 3650 50  0001 C CNN
@@
 $EndComp
 $Comp
-L Conn_01x03 P20
+L Conn_01x03 P402
 U 1 1 5A00395B
 P 6850 3650
-F 0 "P20" H 6850 3850 50  0000 C CNN
+F 0 "P402" H 6850 3850 50  0000 C CNN
 F 1 "CAN_IO" H 6850 3450 50  0000 C CNN
 F 2 "" H 6850 3650 50  0001 C CNN

Commit message: Setting the schematic's footprints.
Parts:
- C401: footprint (none) -> Capacitors_SMD:C_1206_HandSoldering
- P401, P402: footprint (none) -> Connectors_Molex:Molex_KK-6410-03_03x2.54mm_Straight
- U401: footprint (none) -> xenocad.housings:SOIC-8_3.9x4.9mm_Pitch1.27mm
Changed lines of the file:
@@
 F 0 "U401" H 5550 4350 50  0000 R CNN
 F 1 "SN65HVD232" H 5550 4250 50  0000 R CNN
-F 2 "" H 5650 3450 50  0001 C CNN
+F 2 "xenocad.housings:SOIC-8_3.9x4.9mm_Pitch1.27mm" H 5650 3450 50  0001 C CNN
 F 3 "" H 5550 4350 50  0001 C CNN
 	1    5650 3950
@@
 F 0 "C401" H 4825 4400 50  0000 L CNN
 F 1 "100nF" H 4825 4200 50  0000 L CNN
-F 2 "" H 4838 4150 50  0001 C CNN
+F 2 "Capacitors_SMD:C_1206_HandSoldering" H 4838 4150 50  0001 C CNN
 F 3 "" H 4800 4300 50  0001 C CNN
 	1    4800 4300
@@
 F 0 "P401" H 6350 3850 50  0000 C CNN
 F 1 "CAN_IO" H 6350 3450 50  0000 C CNN
-F 2 "" H 6350 3650 50  0001 C CNN
+F 2 "Connectors_Molex:Molex_KK-6410-03_03x2.54mm_Straight" H 6350 3650 50  0001 C CNN
 F 3 "" H 6350 3650 50  0001 C CNN
 	1    6350 3650
@@
 F 0 "P402" H 6850 3850 50  0000 C CNN
 F 1 "CAN_IO" H 6850 3450 50  0000 C CNN
-F 2 "" H 6850 3650 50  0001 C CNN
+F 2 "Connectors_Molex:Molex_KK-6410-03_03x2.54mm_Straight" H 6850 3650 50  0001 C CNN
 F 3 "" H 6850 3650 50  0001 C CNN
 	1    6850 3650
