File: DebouncedInput.sch (KiCad schematic (older format))
At the start: 4 parts, among them P14 Input

Commit message: Changing some value fields on the schematics for a better grouped_csv BOM generation.
Parts:
- P14: value Input -> DebouncedInput_IO
Changed lines of the file:
@@
 AR Path="/59FFBA2E/5603CA46" Ref="P18"  Part="1"
 F 0 "P18" H 5500 4050 50  0000 C CNN
-F 1 "Input" V 5600 3850 50  0000 C CNN
+F 1 "DebouncedInput_IO" V 5600 3850 50  0000 C CNN
 F 2 "" H 5500 3900 60  0001 C CNN
 F 3 "" H 5500 3900 60  0000 C CNN

Commit message: Updating the schematic's annotations.
Parts:
- renumbered C24 to C1401, P14 to P1401, R32 to R1401, R33 to R1402
Changed lines of the file:
@@
 $EndDescr
 $Comp
-L R R32
+L R R1401
 U 1 1 5603CA31
 P 5700 3350
-AR Path="/59FB8E3B/5603CA31" Ref="R32"  Part="1"
-AR Path="/59FFA84C/5603CA31" Ref="R34"  Part="1"
-AR Path="/59FFAD62/5603CA31" Ref="R36"  Part="1"
-AR Path="/59FFAD67/5603CA31" Ref="R38"  Part="1"
-AR Path="/59FFBA2E/5603CA31" Ref="R40"  Part="1"
-F 0 "R40" V 5780 3350 50  0000 C CNN
+AR Path="/59FB8E3B/5603CA31" Ref="R1401"  Part="1"
+AR Path="/59FFA84C/5603CA31" Ref="R1501"  Part="1"
+AR Path="/59FFAD62/5603CA31" Ref="R1601"  Part="1"
+AR Path="/59FFAD67/5603CA31" Ref="R1701"  Part="1"
+AR Path="/59FFBA2E/5603CA31" Ref="R1801"  Part="1"
+F 0 "R1801" V 5780 3350 50  0000 C CNN
 F 1 "100kΩ" V 5700 3350 50  0000 C CNN
 F 2 "" V 5630 3350 30  0001 C CNN
@@
 $EndComp
 $Comp
-L R R33
+L R R1402
 U 1 1 5603CA38
 P 5950 3500
-AR Path="/59FB8E3B/5603CA38" Ref="R33"  Part="1"
-AR Path="/59FFA84C/5603CA38" Ref="R35"  Part="1"
-AR Path="/59FFAD62/5603CA38" Ref="R37"  Part="1"
-AR Path="/59FFAD67/5603CA38" Ref="R39"  Part="1"
-AR Path="/59FFBA2E/5603CA38" Ref="R41"  Part="1"
-F 0 "R41" V 6030 3500 50  0000 C CNN
+AR Path="/59FB8E3B/5603CA38" Ref="R1402"  Part="1"
+AR Path="/59FFA84C/5603CA38" Ref="R1502"  Part="1"
+AR Path="/59FFAD62/5603CA38" Ref="R1602"  Part="1"
+AR Path="/59FFAD67/5603CA38" Ref="R1702"  Part="1"
+AR Path="/59FFBA2E/5603CA38" Ref="R1802"  Part="1"
+F 0 "R1802" V 6030 3500 50  0000 C CNN
 F 1 "18kΩ" V 5950 3500 50  0000 C CNN
 F 2 "" V 5880 3500 30  0001 C CNN
@@
 $EndComp
 $Comp
-L C C24
+L C C1401
 U 1 1 5603CA3F
 P 6150 3750
-AR Path="/59FB8E3B/5603CA3F" Ref="C24"  Part="1"
-AR Path="/59FFA84C/5603CA3F" Ref="C25"  Part="1"
-AR Path="/59FFAD62/5603CA3F" Ref="C26"  Part="1"
-AR Path="/59FFAD67/5603CA3F" Ref="C27"  Part="1"
-AR Path="/59FFBA2E/5603CA3F" Ref="C28"  Part="1"
-F 0 "C28" H 6175 3850 50  0000 L CNN
+AR Path="/59FB8E3B/5603CA3F" Ref="C1401"  Part="1"
+AR Path="/59FFA84C/5603CA3F" Ref="C1501"  Part="1"
+AR Path="/59FFAD62/5603CA3F" Ref="C1601"  Part="1"
+AR Path="/59FFAD67/5603CA3F" Ref="C1701"  Part="1"
+AR Path="/59FFBA2E/5603CA3F" Ref="C1801"  Part="1"
+F 0 "C1801" H 6175 3850 50  0000 L CNN
 F 1 "1µF" H 6175 3650 50  0000 L CNN
 F 2 "" H 6188 3600 30  0001 C CNN
@@
 $EndComp
 $Comp
-L Conn_01x02 P14
+L Conn_01x02 P1401
 U 1 1 5603CA46
 P 5500 3900
-AR Path="/59FB8E3B/5603CA46" Ref="P14"  Part="1"
-AR Path="/59FFA84C/5603CA46" Ref="P15"  Part="1"
-AR Path="/59FFAD62/5603CA46" Ref="P16"  Part="1"
-AR Path="/59FFAD67/5603CA46" Ref="P17"  Part="1"
-AR Path="/59FFBA2E/5603CA46" Ref="P18"  Part="1"
-F 0 "P18" H 5500 4050 50  0000 C CNN
+AR Path="/59FB8E3B/5603CA46" Ref="P1401"  Part="1"
+AR Path="/59FFA84C/5603CA46" Ref="P1501"  Part="1"
+AR Path="/59FFAD62/5603CA46" Ref="P1601"  Part="1"
+AR Path="/59FFAD67/5603CA46" Ref="P1701"  Part="1"
+AR Path="/59FFBA2E/5603CA46" Ref="P1801"  Part="1"
+F 0 "P1801" H 5500 4050 50  0000 C CNN
 F 1 "DebouncedInput_IO" V 5600 3850 50  0000 C CNN
 F 2 "" H 5500 3900 60  0001 C CNN

Commit message: Setting the schematic's footprints.
Parts:
- C1401: footprint (none) -> Capacitors_SMD:C_1206_HandSoldering
- P1401: footprint (none) -> Connectors_Molex:Molex_KK-6410-02_02x2.54mm_Straight
- R1401, R1402: footprint (none) -> Resistors_SMD:R_1206_HandSoldering
Changed lines of the file:
@@
 F 0 "R1801" V 5780 3350 50  0000 C CNN
 F 1 "100kΩ" V 5700 3350 50  0000 C CNN
-F 2 "" V 5630 3350 30  0001 C CNN
+F 2 "Resistors_SMD:R_1206_HandSoldering" V 5630 3350 30  0001 C CNN
 F 3 "" H 5700 3350 30  0000 C CNN
 	1    5700 3350
@@
 F 0 "R1802" V 6030 3500 50  0000 C CNN
 F 1 "18kΩ" V 5950 3500 50  0000 C CNN
-F 2 "" V 5880 3500 30  0001 C CNN
+F 2 "Resistors_SMD:R_1206_HandSoldering" V 5880 3500 30  0001 C CNN
 F 3 "" H 5950 3500 30  0000 C CNN
 	1    5950 3500
@@
 F 0 "C1801" H 6175 3850 50  0000 L CNN
 F 1 "1µF" H 6175 3650 50  0000 L CNN
-F 2 "" H 6188 3600 30  0001 C CNN
+F 2 "Capacitors_SMD:C_1206_HandSoldering" H 6188 3600 30  0001 C CNN
 F 3 "" H 6150 3750 60  0000 C CNN
 	1    6150 3750
@@
 F 0 "P1801" H 5500 4050 50  0000 C CNN
 F 1 "DebouncedInput_IO" V 5600 3850 50  0000 C CNN
-F 2 "" H 5500 3900 60  0001 C CNN
+F 2 "Connectors_Molex:Molex_KK-6410-02_02x2.54mm_Straight" H 5500 3900 60  0001 C CNN
 F 3 "" H 5500 3900 60  0000 C CNN
 	1    5500 3900
