File: Driver.sch (KiCad schematic (older format))
At the start: 10 parts, among them P12 Motor, U1 LMD18201

Commit message: Adding Hermes 2 schematic files.
Parts:
- removed C13: 1nF, Footprints:C_CMS0603, symbol C
- removed C14, C15: 10nF, Footprints:C_CMS0603, symbol C
- removed CP1: 330µF, Footprints:C_Radial, symbol CP1
- removed P12: Motor, Footprints:Power_Conn_01x02, symbol CONN_01X02
- removed R24, R25: 10kΩ, Footprints:R_CMS1206, symbol R
- removed U1: LMD18201, Footprints:LMD18201, symbol LMD18201
- added C6: 10µF, symbol C
- added C7: 100nF, symbol C
- added Carrier1: Pololu_Dual_VNHxSP30_Motor_Driver_Carrier, symbol Pololu_Dual_VNHxSP30_Motor_Driver_Carrier
- C8: renamed from C12; footprint Footprints:C_CMS1210 -> (none)
- C9: renamed from C11; footprint Footprints:C_CMS0603 -> (none)
Connections:
- net labels added: +5V, CS_1, CS_2, DIAG_1, DIAG_2, IN_A_1, IN_A_2, IN_B_1, IN_B_2, PWM_1, PWM_2
- net labels removed: Direction, PWM, ThermalFlag
- wire segments 29 -> 6
Other:
- note added: "Two 330µF electrolytic capacitors are\nalready soldered on the carrier."
- moved on the sheet: C8, C9

Commit message: Updating the schematic's annotations.
Parts:
- renumbered C6 to C501, C7 to C502, C8 to C503, C9 to C504, Carrier1 to Carrier501
Changed lines of the file:
@@
 GND
 $Comp
-L C C9
+L C C504
 U 1 1 55E9687D
 P 8400 3950
-F 0 "C9" H 8425 4050 50  0000 L CNN
+F 0 "C504" H 8425 4050 50  0000 L CNN
 F 1 "100nF" H 8425 3850 50  0000 L CNN
 F 2 "" H 8438 3800 30  0001 C CNN
@@
 $EndComp
 $Comp
-L C C8
+L C C503
 U 1 1 55E968B0
 P 8100 3950
-F 0 "C8" H 8125 4050 50  0000 L CNN
+F 0 "C503" H 8125 4050 50  0000 L CNN
 F 1 "10µF" H 8125 3850 50  0000 L CNN
 F 2 "" H 8138 3800 30  0001 C CNN
@@
 +5V
 $Comp
-L C C7
+L C C502
 U 1 1 59FB935D
 P 7800 3950
-F 0 "C7" H 7825 4050 50  0000 L CNN
+F 0 "C502" H 7825 4050 50  0000 L CNN
 F 1 "100nF" H 7825 3850 50  0000 L CNN
 F 2 "" H 7838 3800 30  0001 C CNN
@@
 $EndComp
 $Comp
-L C C6
+L C C501
 U 1 1 59FB9363
 P 7500 3950
-F 0 "C6" H 7525 4050 50  0000 L CNN
+F 0 "C501" H 7525 4050 50  0000 L CNN
 F 1 "10µF" H 7525 3850 50  0000 L CNN
 F 2 "" H 7538 3800 30  0001 C CNN
@@
 $EndComp
 $Comp
-L Pololu_Dual_VNHxSP30_Motor_Driver_Carrier Carrier1
+L Pololu_Dual_VNHxSP30_Motor_Driver_Carrier Carrier501
 U 1 1 59FBA21B
 P 5900 3950
-F 0 "Carrier1" H 5900 5150 60  0000 C CNN
+F 0 "Carrier501" H 5900 5150 60  0000 C CNN
 F 1 "Pololu_Dual_VNHxSP30_Motor_Driver_Carrier" H 5900 5000 60  0000 C CNN
 F 2 "" H 5900 4300 60  0001 C CNN

Commit message: Setting the schematic's footprints.
Parts:
- C501, C502, C503, C504: footprint (none) -> Capacitors_SMD:C_1206_HandSoldering
- Carrier501: footprint (none) -> xenocad.motor_driver:Pololu_Dual_VNHxSP30_Motor_Driver_no_output
Changed lines of the file:
@@
 F 0 "C504" H 8425 4050 50  0000 L CNN
 F 1 "100nF" H 8425 3850 50  0000 L CNN
-F 2 "" H 8438 3800 30  0001 C CNN
+F 2 "Capacitors_SMD:C_1206_HandSoldering" H 8438 3800 30  0001 C CNN
 F 3 "" H 8400 3950 60  0000 C CNN
 	1    8400 3950
@@
 F 0 "C503" H 8125 4050 50  0000 L CNN
 F 1 "10µF" H 8125 3850 50  0000 L CNN
-F 2 "" H 8138 3800 30  0001 C CNN
+F 2 "Capacitors_SMD:C_1206_HandSoldering" H 8138 3800 30  0001 C CNN
 F 3 "" H 8100 3950 60  0000 C CNN
 	1    8100 3950
@@
 F 0 "C502" H 7825 4050 50  0000 L CNN
 F 1 "100nF" H 7825 3850 50  0000 L CNN
-F 2 "" H 7838 3800 30  0001 C CNN
+F 2 "Capacitors_SMD:C_1206_HandSoldering" H 7838 3800 30  0001 C CNN
 F 3 "" H 7800 3950 60  0000 C CNN
 	1    7800 3950
@@
 F 0 "C501" H 7525 4050 50  0000 L CNN
 F 1 "10µF" H 7525 3850 50  0000 L CNN
-F 2 "" H 7538 3800 30  0001 C CNN
+F 2 "Capacitors_SMD:C_1206_HandSoldering" H 7538 3800 30  0001 C CNN
 F 3 "" H 7500 3950 60  0000 C CNN
 	1    7500 3950
@@
 F 0 "Carrier501" H 5900 5150 60  0000 C CNN
 F 1 "Pololu_Dual_VNHxSP30_Motor_Driver_Carrier" H 5900 5000 60  0000 C CNN
-F 2 "" H 5900 4300 60  0001 C CNN
+F 2 "xenocad.motor_driver:Pololu_Dual_VNHxSP30_Motor_Driver_no_output" H 5900 4300 60  0001 C CNN
 F 3 "" H 5900 4300 60  0001 C CNN
 	1    5900 3950
