File: Encoder.sch (KiCad schematic (older format))
At the start: 6 parts, among them P7 Encoder

Commit message: Adding Hermes 2 schematic files.
Parts:
- C10: renamed from C9; footprint Footprints:C_CMS0603 -> (none)
- P6: renamed from P7; footprint Footprints:Conn_01x04 -> (none); symbol CONN_01X04 -> Conn_01x04
- R12: renamed from R10; footprint Footprints:R_CMS1206 -> (none)
- R13: renamed from R11; footprint Footprints:R_CMS1206 -> (none)
- R14: renamed from R12; footprint Footprints:R_CMS1206 -> (none)
- R15: renamed from R13; footprint Footprints:R_CMS1206 -> (none)
Changed lines of the file:
@@
 EESchema Schematic File Version 2
-LIBS:power
 LIBS:device
-LIBS:transistors
 LIBS:conn
-LIBS:linear
-LIBS:regul
-LIBS:74xx
-LIBS:cmos4000
-LIBS:adc-dac
-LIBS:memory
-LIBS:xilinx
-LIBS:microcontrollers
-LIBS:dsp
-LIBS:microchip
-LIBS:analog_switches
-LIBS:motorola
-LIBS:texas
-LIBS:intel
-LIBS:audio
-LIBS:interface
-LIBS:digital-audio
-LIBS:philips
-LIBS:display
-LIBS:cypress
-LIBS:siliconi
-LIBS:opto
-LIBS:atmel
-LIBS:contrib
-LIBS:valves
-LIBS:Hermes-cache
 EELAYER 25 0
 EELAYER END
 $Descr A4 11693 8268
 encoding utf-8
-Sheet 7 17
-Title ""
+Sheet 6 18
+Title "Encoder"
 Date ""
-Rev ""
+Rev "rev1"
 Comp ""
 Comment1 ""
@@
 $EndDescr
 $Comp
-L CONN_01X04 P7
+L Conn_01x04 P6
 U 1 1 55E71CE3
-P 5850 4300
-AR Path="/55E78073/55E71CE3" Ref="P7"  Part="1"
-AR Path="/55E78AE8/55E71CE3" Ref="P8"  Part="1"
-F 0 "P7" H 5850 4550 50  0000 C CNN
-F 1 "Encoder" V 5950 4300 50  0000 C CNN
-F 2 "Footprints:Conn_01x04" H 5850 4300 60  0001 C CNN
-F 3 "" H 5850 4300 60  0000 C CNN
-	1    5850 4300
+P 5900 4300
+AR Path="/59FB8F5F/55E71CE3" Ref="P6"  Part="1"
+AR Path="/59FF91FA/55E71CE3" Ref="P7"  Part="1"
+F 0 "P7" H 5900 4550 50  0000 C CNN
+F 1 "Encoder" V 6000 4250 50  0000 C CNN
+F 2 "" H 5900 4300 60  0001 C CNN
+F 3 "" H 5900 4300 60  0000 C CNN
+	1    5900 4300
 	0    1    1    0
 $EndComp
 $Comp
-L C C9
+L C C10
 U 1 1 55E71CEC
 P 6800 3950
-AR Path="/55E78073/55E71CEC" Ref="C9"  Part="1"
-AR Path="/55E78AE8/55E71CEC" Ref="C10"  Part="1"
-F 0 "C9" H 6825 4050 50  0000 L CNN
+AR Path="/59FB8F5F/55E71CEC" Ref="C10"  Part="1"
+AR Path="/59FF91FA/55E71CEC" Ref="C11"  Part="1"
+F 0 "C11" H 6825 4050 50  0000 L CNN
 F 1 "100nF" H 6825 3850 50  0000 L CNN
-F 2 "Footprints:C_CMS0603" H 6838 3800 30  0001 C CNN
+F 2 "" H 6838 3800 30  0001 C CNN
 F 3 "" H 6800 3950 60  0000 C CNN
 	1    6800 3950
@@
 B
 $Comp
-L R R10
+L R R12
 U 1 1 5602AF11
 P 5600 3200
-AR Path="/55E78073/5602AF11" Ref="R10"  Part="1"
-AR Path="/55E78AE8/5602AF11" Ref="R14"  Part="1"
-F 0 "R10" V 5680 3200 50  0000 C CNN
+AR Path="/59FB8F5F/5602AF11" Ref="R12"  Part="1"
+AR Path="/59FF91FA/5602AF11" Ref="R16"  Part="1"
+F 0 "R16" V 5680 3200 50  0000 C CNN
 F 1 "22Ω" V 5600 3200 50  0000 C CNN
-F 2 "Footprints:R_CMS1206" V 5530 3200 30  0001 C CNN
+F 2 "" V 5530 3200 30  0001 C CNN
 F 3 "" H 5600 3200 30  0000 C CNN
 	1    5600 3200
@@
 $EndComp
 $Comp
-L R R11
+L R R13
 U 1 1 5602AF44
 P 5900 3200
-AR Path="/55E78073/5602AF44" Ref="R11"  Part="1"
-AR Path="/55E78AE8/5602AF44" Ref="R15"  Part="1"
-F 0 "R11" V 5980 3200 50  0000 C CNN
+AR Path="/59FB8F5F/5602AF44" Ref="R13"  Part="1"
+AR Path="/59FF91FA/5602AF44" Ref="R17"  Part="1"
+F 0 "R17" V 5980 3200 50  0000 C CNN
 F 1 "22Ω" V 5900 3200 50  0000 C CNN
-F 2 "Footprints:R_CMS1206" V 5830 3200 30  0001 C CNN
+F 2 "" V 5830 3200 30  0001 C CNN
 F 3 "" H 5900 3200 30  0000 C CNN
 	1    5900 3200
@@
 $EndComp
 $Comp
-L R R13
+L R R15
 U 1 1 5602B19C
 P 6350 3650
-AR Path="/55E78073/5602B19C" Ref="R13"  Part="1"
-AR Path="/55E78AE8/5602B19C" Ref="R17"  Part="1"
-F 0 "R13" V 6430 3650 50  0000 C CNN
+AR Path="/59FB8F5F/5602B19C" Ref="R15"  Part="1"
+AR Path="/59FF91FA/5602B19C" Ref="R19"  Part="1"
+F 0 "R19" V 6430 3650 50  0000 C CNN
 F 1 "10kΩ" V 6350 3650 50  0000 C CNN
-F 2 "Footprints:R_CMS1206" V 6280 3650 30  0001 C CNN
+F 2 "" V 6280 3650 30  0001 C CNN
 F 3 "" H 6350 3650 30  0000 C CNN
 	1    6350 3650
@@
 $EndComp
 $Comp
-L R R12
+L R R14
 U 1 1 5602B1C5
 P 6350 3450
-AR Path="/55E78073/5602B1C5" Ref="R12"  Part="1"
-AR Path="/55E78AE8/5602B1C5" Ref="R16"  Part="1"
-F 0 "R12" V 6430 3450 50  0000 C CNN
+AR Path="/59FB8F5F/5602B1C5" Ref="R14"  Part="1"
+AR Path="/59FF91FA/5602B1C5" Ref="R18"  Part="1"
+F 0 "R18" V 6430 3450 50  0000 C CNN
 F 1 "10kΩ" V 6350 3450 50  0000 C CNN
-F 2 "Footprints:R_CMS1206" V 6280 3450 30  0001 C CNN
+F 2 "" V 6280 3450 30  0001 C CNN
 F 3 "" H 6350 3450 30  0000 C CNN
 	1    6350 3450

Commit message: Rearranging encoder sheet so GND is at the bottom and power supply at the top.
Connections:
- wire segments 15 -> 20
Other:
- moved on the sheet: C10, R14, R15
Changed lines of the file:
@@
 AR Path="/59FB8F5F/55E71CE3" Ref="P6"  Part="1"
 AR Path="/59FF91FA/55E71CE3" Ref="P7"  Part="1"
-F 0 "P7" H 5900 4550 50  0000 C CNN
+F 0 "P6" H 5900 4550 50  0000 C CNN
 F 1 "Encoder" V 6000 4250 50  0000 C CNN
 F 2 "" H 5900 4300 60  0001 C CNN
@@
 L C C10
 U 1 1 55E71CEC
-P 6800 3950
+P 6600 3750
 AR Path="/59FB8F5F/55E71CEC" Ref="C10"  Part="1"
 AR Path="/59FF91FA/55E71CEC" Ref="C11"  Part="1"
-F 0 "C11" H 6825 4050 50  0000 L CNN
-F 1 "100nF" H 6825 3850 50  0000 L CNN
-F 2 "" H 6838 3800 30  0001 C CNN
-F 3 "" H 6800 3950 60  0000 C CNN
-	1    6800 3950
+F 0 "C10" H 6625 3850 50  0000 L CNN
+F 1 "100nF" H 6625 3650 50  0000 L CNN
+F 2 "" H 6638 3600 30  0001 C CNN
+F 3 "" H 6600 3750 60  0000 C CNN
+	1    6600 3750
 	1    0    0    -1
 $EndComp
-Text HLabel 6800 4300 3    60   Input ~ 0
+Text HLabel 6650 3400 1    60   Input ~ 0
 +5V
-Text HLabel 6800 3000 1    60   Input ~ 0
+Text HLabel 6650 4100 3    60   Input ~ 0
 GND
 Text HLabel 5900 3000 1    60   Output ~ 0
@@
 AR Path="/59FB8F5F/5602AF11" Ref="R12"  Part="1"
 AR Path="/59FF91FA/5602AF11" Ref="R16"  Part="1"
-F 0 "R16" V 5680 3200 50  0000 C CNN
+F 0 "R12" V 5680 3200 50  0000 C CNN
 F 1 "22Ω" V 5600 3200 50  0000 C CNN
 F 2 "" V 5530 3200 30  0001 C CNN
@@
 AR Path="/59FB8F5F/5602AF44" Ref="R13"  Part="1"
 AR Path="/59FF91FA/5602AF44" Ref="R17"  Part="1"
-F 0 "R17" V 5980 3200 50  0000 C CNN
+F 0 "R13" V 5980 3200 50  0000 C CNN
 F 1 "22Ω" V 5900 3200 50  0000 C CNN
 F 2 "" V 5830 3200 30  0001 C CNN
@@
 L R R15
 U 1 1 5602B19C
-P 6350 3650
+P 6400 3750
 AR Path="/59FB8F5F/5602B19C" Ref="R15"  Part="1"
 AR Path="/59FF91FA/5602B19C" Ref="R19"  Part="1"
-F 0 "R19" V 6430 3650 50  0000 C CNN
-F 1 "10kΩ" V 6350 3650 50  0000 C CNN
-F 2 "" V 6280 3650 30  0001 C CNN
-F 3 "" H 6350 3650 30  0000 C CNN
-	1    6350 3650
-	0    1    1    0
+F 0 "R15" V 6480 3750 50  0000 C CNN
+F 1 "10kΩ" V 6400 3750 50  0000 C CNN
+F 2 "" V 6330 3750 30  0001 C CNN
+F 3 "" H 6400 3750 30  0000 C CNN
+	1    6400 3750
+	-1   0    0    1
 $EndComp
 $Comp
 L R R14
 U 1 1 5602B1C5
-P 6350 3450
+P 6200 3800
 AR Path="/59FB8F5F/5602B1C5" Ref="R14"  Part="1"
 AR Path="/59FF91FA/5602B1C5" Ref="R18"  Part="1"
-F 0 "R18" V 6430 3450 50  0000 C CNN
-F 1 "10kΩ" V 6350 3450 50  0000 C CNN
-F 2 "" V 6280 3450 30  0001 C CNN
-F 3 "" H 6350 3450 30  0000 C CNN
-	1    6350 3450
-	0    1    1    0
+F 0 "R14" V 6280 3800 50  0000 C CNN
+F 1 "10kΩ" V 6200 3800 50  0000 C CNN
+F 2 "" V 6130 3800 30  0001 C CNN
+F 3 "" H 6200 3800 30  0000 C CNN
+	1    6200 3800
+	-1   0    0    1
 $EndComp
-Wire Wire Line
-	6000 4100 6800 4100
-Wire Wire Line
-	5900 4100 5900 3800
-Wire Wire Line
-	5900 3800 6800 3800
 Wire Wire Line
 	5800 3350 5800 4100
@@
 	5700 3350 5700 4100
 Wire Wire Line
-	6800 3800 6800 3000
-Wire Wire Line
-	6500 3650 6800 3650
-Connection ~ 6800 3650
-Wire Wire Line
-	6500 3450 6800 3450
-Connection ~ 6800 3450
-Wire Wire Line
-	5800 3650 6200 3650
-Wire Wire Line
-	5700 3450 6200 3450
-Wire Wire Line
 	5800 3350 5900 3350
-Connection ~ 5800 3650
 Wire Wire Line
 	5700 3350 5600 3350
-Connection ~ 5700 3450
 Wire Wire Line
 	5900 3050 5900 3000
@@
 	5600 3050 5600 3000
 Wire Wire Line
-	6800 4100 6800 4300
+	5900 4100 5900 4000
+Wire Wire Line
+	5900 4000 6650 4000
+Wire Wire Line
+	6650 4000 6650 4100
+Wire Wire Line
+	6600 3900 6600 4000
+Connection ~ 6600 4000
+Wire Wire Line
+	6400 3900 6400 4000
+Connection ~ 6400 4000
+Wire Wire Line
+	6200 3950 6200 4000
+Connection ~ 6200 4000
+Wire Wire Line
+	6000 3500 6000 4100
+Wire Wire Line
+	6000 3500 6650 3500
+Wire Wire Line
+	6650 3500 6650 3400
+Wire Wire Line
+	6600 3600 6600 3500
+Connection ~ 6600 3500
+Wire Wire Line
+	6200 3650 6200 3600
+Wire Wire Line
+	6200 3600 5700 3600
+Connection ~ 5700 3600
+Wire Wire Line
+	5800 3550 6400 3550
+Wire Wire Line
+	6400 3550 6400 3600
+Connection ~ 5800 3550
 $EndSCHEMATC

Commit message: Changing some value fields on the schematics for a better grouped_csv BOM generation.
Parts:
- P6: value Encoder -> Encoder_IO
Changed lines of the file:
@@
 AR Path="/59FF91FA/55E71CE3" Ref="P7"  Part="1"
 F 0 "P6" H 5900 4550 50  0000 C CNN
-F 1 "Encoder" V 6000 4250 50  0000 C CNN
+F 1 "Encoder_IO" V 6000 4250 50  0000 C CNN
 F 2 "" H 5900 4300 60  0001 C CNN
 F 3 "" H 5900 4300 60  0000 C CNN

Commit message: Updating the schematic's annotations.
Parts:
- renumbered C10 to C601, P6 to P601, R12 to R601, R13 to R602, R14 to R603, R15 to R604
Changed lines of the file:
@@
 $EndDescr
 $Comp
-L Conn_01x04 P6
+L Conn_01x04 P601
 U 1 1 55E71CE3
 P 5900 4300
-AR Path="/59FB8F5F/55E71CE3" Ref="P6"  Part="1"
-AR Path="/59FF91FA/55E71CE3" Ref="P7"  Part="1"
-F 0 "P6" H 5900 4550 50  0000 C CNN
+AR Path="/59FB8F5F/55E71CE3" Ref="P601"  Part="1"
+AR Path="/59FF91FA/55E71CE3" Ref="P701"  Part="1"
+F 0 "P701" H 5900 4550 50  0000 C CNN
 F 1 "Encoder_IO" V 6000 4250 50  0000 C CNN
 F 2 "" H 5900 4300 60  0001 C CNN
@@
 $EndComp
 $Comp
-L C C10
+L C C601
 U 1 1 55E71CEC
 P 6600 3750
-AR Path="/59FB8F5F/55E71CEC" Ref="C10"  Part="1"
-AR Path="/59FF91FA/55E71CEC" Ref="C11"  Part="1"
-F 0 "C10" H 6625 3850 50  0000 L CNN
+AR Path="/59FB8F5F/55E71CEC" Ref="C601"  Part="1"
+AR Path="/59FF91FA/55E71CEC" Ref="C701"  Part="1"
+F 0 "C701" H 6625 3850 50  0000 L CNN
 F 1 "100nF" H 6625 3650 50  0000 L CNN
 F 2 "" H 6638 3600 30  0001 C CNN
@@
 B
 $Comp
-L R R12
+L R R601
 U 1 1 5602AF11
 P 5600 3200
-AR Path="/59FB8F5F/5602AF11" Ref="R12"  Part="1"
-AR Path="/59FF91FA/5602AF11" Ref="R16"  Part="1"
-F 0 "R12" V 5680 3200 50  0000 C CNN
+AR Path="/59FB8F5F/5602AF11" Ref="R601"  Part="1"
+AR Path="/59FF91FA/5602AF11" Ref="R701"  Part="1"
+F 0 "R701" V 5680 3200 50  0000 C CNN
 F 1 "22Ω" V 5600 3200 50  0000 C CNN
 F 2 "" V 5530 3200 30  0001 C CNN
@@
 $EndComp
 $Comp
-L R R13
+L R R602
 U 1 1 5602AF44
 P 5900 3200
-AR Path="/59FB8F5F/5602AF44" Ref="R13"  Part="1"
-AR Path="/59FF91FA/5602AF44" Ref="R17"  Part="1"
-F 0 "R13" V 5980 3200 50  0000 C CNN
+AR Path="/59FB8F5F/5602AF44" Ref="R602"  Part="1"
+AR Path="/59FF91FA/5602AF44" Ref="R702"  Part="1"
+F 0 "R702" V 5980 3200 50  0000 C CNN
 F 1 "22Ω" V 5900 3200 50  0000 C CNN
 F 2 "" V 5830 3200 30  0001 C CNN
@@
 $EndComp
 $Comp
-L R R15
+L R R604
 U 1 1 5602B19C
 P 6400 3750
-AR Path="/59FB8F5F/5602B19C" Ref="R15"  Part="1"
-AR Path="/59FF91FA/5602B19C" Ref="R19"  Part="1"
-F 0 "R15" V 6480 3750 50  0000 C CNN
+AR Path="/59FB8F5F/5602B19C" Ref="R604"  Part="1"
+AR Path="/59FF91FA/5602B19C" Ref="R704"  Part="1"
+F 0 "R704" V 6480 3750 50  0000 C CNN
 F 1 "10kΩ" V 6400 3750 50  0000 C CNN
 F 2 "" V 6330 3750 30  0001 C CNN
@@
 $EndComp
 $Comp
-L R R14
+L R R603
 U 1 1 5602B1C5
 P 6200 3800
-AR Path="/59FB8F5F/5602B1C5" Ref="R14"  Part="1"
-AR Path="/59FF91FA/5602B1C5" Ref="R18"  Part="1"
-F 0 "R14" V 6280 3800 50  0000 C CNN
+AR Path="/59FB8F5F/5602B1C5" Ref="R603"  Part="1"
+AR Path="/59FF91FA/5602B1C5" Ref="R703"  Part="1"
+F 0 "R703" V 6280 3800 50  0000 C CNN
 F 1 "10kΩ" V 6200 3800 50  0000 C CNN
 F 2 "" V 6130 3800 30  0001 C CNN

Commit message: Setting the schematic's footprints.
Parts:
- C601: footprint (none) -> Capacitors_SMD:C_1206_HandSoldering
- P601: footprint (none) -> Connectors_Molex:Molex_KK-6410-04_04x2.54mm_Straight
- R601, R602, R603, R604: footprint (none) -> Resistors_SMD:R_1206_HandSoldering
Changed lines of the file:
@@
 F 0 "P701" H 5900 4550 50  0000 C CNN
 F 1 "Encoder_IO" V 6000 4250 50  0000 C CNN
-F 2 "" H 5900 4300 60  0001 C CNN
+F 2 "Connectors_Molex:Molex_KK-6410-04_04x2.54mm_Straight" H 5900 4300 60  0001 C CNN
 F 3 "" H 5900 4300 60  0000 C CNN
 	1    5900 4300
@@
 F 0 "C701" H 6625 3850 50  0000 L CNN
 F 1 "100nF" H 6625 3650 50  0000 L CNN
-F 2 "" H 6638 3600 30  0001 C CNN
+F 2 "Capacitors_SMD:C_1206_HandSoldering" H 6638 3600 30  0001 C CNN
 F 3 "" H 6600 3750 60  0000 C CNN
 	1    6600 3750
@@
 F 0 "R701" V 5680 3200 50  0000 C CNN
 F 1 "22Ω" V 5600 3200 50  0000 C CNN
-F 2 "" V 5530 3200 30  0001 C CNN
+F 2 "Resistors_SMD:R_1206_HandSoldering" V 5530 3200 30  0001 C CNN
 F 3 "" H 5600 3200 30  0000 C CNN
 	1    5600 3200
@@
 F 0 "R702" V 5980 3200 50  0000 C CNN
 F 1 "22Ω" V 5900 3200 50  0000 C CNN
-F 2 "" V 5830 3200 30  0001 C CNN
+F 2 "Resistors_SMD:R_1206_HandSoldering" V 5830 3200 30  0001 C CNN
 F 3 "" H 5900 3200 30  0000 C CNN
 	1    5900 3200
@@
 F 0 "R704" V 6480 3750 50  0000 C CNN
 F 1 "10kΩ" V 6400 3750 50  0000 C CNN
-F 2 "" V 6330 3750 30  0001 C CNN
+F 2 "Resistors_SMD:R_1206_HandSoldering" V 6330 3750 30  0001 C CNN
 F 3 "" H 6400 3750 30  0000 C CNN
 	1    6400 3750
@@
 F 0 "R703" V 6280 3800 50  0000 C CNN
 F 1 "10kΩ" V 6200 3800 50  0000 C CNN
-F 2 "" V 6130 3800 30  0001 C CNN
+F 2 "Resistors_SMD:R_1206_HandSoldering" V 6130 3800 30  0001 C CNN
 F 3 "" H 6200 3800 30  0000 C CNN
 	1    6200 3800
