File: GP2.sch (KiCad schematic (older format))
At the start: 5 parts, among them P1 GP2

Commit message: Adding Hermes 2 schematic files.
Parts:
- C12: renamed from C1; footprint Footprints:C_CMS1210 -> (none)
- C13: renamed from C2; footprint Footprints:C_CMS0603 -> (none)
- P8: renamed from P1; footprint Footprints:Conn_01x03 -> (none); symbol CONN_01X03 -> Conn_01x03
- R20: renamed from R2; footprint Footprints:R_CMS1206 -> (none)
- R21: renamed from R3; footprint Footprints:R_CMS1206 -> (none)
Changed lines of the file:
@@
 EESchema Schematic File Version 2
-LIBS:power
 LIBS:device
-LIBS:transistors
 LIBS:conn
-LIBS:linear
-LIBS:regul
-LIBS:74xx
-LIBS:cmos4000
-LIBS:adc-dac
-LIBS:memory
-LIBS:xilinx
-LIBS:microcontrollers
-LIBS:dsp
-LIBS:microchip
-LIBS:analog_switches
-LIBS:motorola
-LIBS:texas
-LIBS:intel
-LIBS:audio
-LIBS:interface
-LIBS:digital-audio
-LIBS:philips
-LIBS:display
-LIBS:cypress
-LIBS:siliconi
-LIBS:opto
-LIBS:atmel
-LIBS:contrib
-LIBS:valves
-LIBS:Hermes-cache
 EELAYER 25 0
 EELAYER END
 $Descr A4 11693 8268
 encoding utf-8
-Sheet 5 17
-Title ""
+Sheet 8 18
+Title "GP2"
 Date ""
-Rev ""
+Rev "rev1"
 Comp ""
-Comment1 ""
+Comment1 "With voltage divider to 3.3V"
 Comment2 ""
 Comment3 ""
@@
 $EndDescr
 $Comp
-L CONN_01X03 P1
+L Conn_01x03 P8
 U 1 1 55E7C054
 P 4900 3750
-AR Path="/55E75835/55E7C054" Ref="P1"  Part="1"
-AR Path="/55E760A5/55E7C054" Ref="P2"  Part="1"
-AR Path="/55E7647A/55E7C054" Ref="P3"  Part="1"
-AR Path="/55E7647F/55E7C054" Ref="P4"  Part="1"
-F 0 "P4" H 4900 3950 50  0000 C CNN
+AR Path="/59FB8CCA/55E7C054" Ref="P8"  Part="1"
+AR Path="/59FF5446/55E7C054" Ref="P9"  Part="1"
+AR Path="/59FF5905/55E7C054" Ref="P10"  Part="1"
+AR Path="/59FF590A/55E7C054" Ref="P11"  Part="1"
+AR Path="/59FF5C5D/55E7C054" Ref="P12"  Part="1"
+AR Path="/59FF5C62/55E7C054" Ref="P13"  Part="1"
+F 0 "P13" H 4900 3950 50  0000 C CNN
 F 1 "GP2" V 5000 3750 50  0000 C CNN
-F 2 "Footprints:Conn_01x03" H 4900 3750 60  0001 C CNN
+F 2 "" H 4900 3750 60  0001 C CNN
 F 3 "" H 4900 3750 60  0000 C CNN
 	1    4900 3750
@@
 $EndComp
 $Comp
-L C C1
+L C C12
 U 1 1 55E7C068
 P 5250 3450
-AR Path="/55E75835/55E7C068" Ref="C1"  Part="1"
-AR Path="/55E760A5/55E7C068" Ref="C3"  Part="1"
-AR Path="/55E7647A/55E7C068" Ref="C5"  Part="1"
-AR Path="/55E7647F/55E7C068" Ref="C7"  Part="1"
-F 0 "C7" H 5275 3550 50  0000 L CNN
+AR Path="/59FB8CCA/55E7C068" Ref="C12"  Part="1"
+AR Path="/59FF5446/55E7C068" Ref="C14"  Part="1"
+AR Path="/59FF5905/55E7C068" Ref="C16"  Part="1"
+AR Path="/59FF590A/55E7C068" Ref="C18"  Part="1"
+AR Path="/59FF5C5D/55E7C068" Ref="C20"  Part="1"
+AR Path="/59FF5C62/55E7C068" Ref="C22"  Part="1"
+F 0 "C22" H 5275 3550 50  0000 L CNN
 F 1 "10µF" H 5275 3350 50  0000 L CNN
-F 2 "Footprints:C_CMS1210" H 5288 3300 30  0001 C CNN
+F 2 "" H 5288 3300 30  0001 C CNN
 F 3 "" H 5250 3450 60  0000 C CNN
 	1    5250 3450
@@
 Signal
 $Comp
-L R R2
+L R R20
 U 1 1 55E88E74
 P 5700 3850
-AR Path="/55E75835/55E88E74" Ref="R2"  Part="1"
-AR Path="/55E760A5/55E88E74" Ref="R4"  Part="1"
-AR Path="/55E7647A/55E88E74" Ref="R6"  Part="1"
-AR Path="/55E7647F/55E88E74" Ref="R8"  Part="1"
-F 0 "R8" V 5780 3850 50  0000 C CNN
+AR Path="/59FB8CCA/55E88E74" Ref="R20"  Part="1"
+AR Path="/59FF5446/55E88E74" Ref="R22"  Part="1"
+AR Path="/59FF5905/55E88E74" Ref="R24"  Part="1"
+AR Path="/59FF590A/55E88E74" Ref="R26"  Part="1"
+AR Path="/59FF5C5D/55E88E74" Ref="R28"  Part="1"
+AR Path="/59FF5C62/55E88E74" Ref="R30"  Part="1"
+F 0 "R30" V 5780 3850 50  0000 C CNN
 F 1 "10kΩ" V 5700 3850 50  0000 C CNN
-F 2 "Footprints:R_CMS1206" V 5630 3850 30  0001 C CNN
+F 2 "" V 5630 3850 30  0001 C CNN
 F 3 "" H 5700 3850 30  0000 C CNN
 	1    5700 3850
@@
 Connection ~ 5950 3850
 $Comp
-L R R3
+L R R21
 U 1 1 55E88FA1
 P 6200 3850
-AR Path="/55E75835/55E88FA1" Ref="R3"  Part="1"
-AR Path="/55E760A5/55E88FA1" Ref="R5"  Part="1"
-AR Path="/55E7647A/55E88FA1" Ref="R7"  Part="1"
-AR Path="/55E7647F/55E88FA1" Ref="R9"  Part="1"
-F 0 "R9" V 6280 3850 50  0000 C CNN
+AR Path="/59FB8CCA/55E88FA1" Ref="R21"  Part="1"
+AR Path="/59FF5446/55E88FA1" Ref="R23"  Part="1"
+AR Path="/59FF5905/55E88FA1" Ref="R25"  Part="1"
+AR Path="/59FF590A/55E88FA1" Ref="R27"  Part="1"
+AR Path="/59FF5C5D/55E88FA1" Ref="R29"  Part="1"
+AR Path="/59FF5C62/55E88FA1" Ref="R31"  Part="1"
+F 0 "R31" V 6280 3850 50  0000 C CNN
 F 1 "20kΩ" V 6200 3850 50  0000 C CNN
-F 2 "Footprints:R_CMS1206" V 6130 3850 30  0001 C CNN
+F 2 "" V 6130 3850 30  0001 C CNN
 F 3 "" H 6200 3850 30  0000 C CNN
 	1    6200 3850
@@
 	6350 3450 5400 3450
 $Comp
-L C C2
+L C C13
 U 1 1 5602AA98
 P 5950 3650
-AR Path="/55E75835/5602AA98" Ref="C2"  Part="1"
-AR Path="/55E760A5/5602AA98" Ref="C4"  Part="1"
-AR Path="/55E7647A/5602AA98" Ref="C6"  Part="1"
-AR Path="/55E7647F/5602AA98" Ref="C8"  Part="1"
-F 0 "C8" H 5975 3750 50  0000 L CNN
+AR Path="/59FB8CCA/5602AA98" Ref="C13"  Part="1"
+AR Path="/59FF5446/5602AA98" Ref="C15"  Part="1"
+AR Path="/59FF5905/5602AA98" Ref="C17"  Part="1"
+AR Path="/59FF590A/5602AA98" Ref="C19"  Part="1"
+AR Path="/59FF5C5D/5602AA98" Ref="C21"  Part="1"
+AR Path="/59FF5C62/5602AA98" Ref="C23"  Part="1"
+F 0 "C23" H 5975 3750 50  0000 L CNN
 F 1 "100nF" H 5975 3550 50  0000 L CNN
-F 2 "Footprints:C_CMS0603" H 5988 3500 30  0001 C CNN
+F 2 "" H 5988 3500 30  0001 C CNN
 F 3 "" H 5950 3650 60  0000 C CNN
 	1    5950 3650

Commit message: Changing some value fields on the schematics for a better grouped_csv BOM generation.
Parts:
- P8: value GP2 -> GP2_IO
Changed lines of the file:
@@
 AR Path="/59FF5C62/55E7C054" Ref="P13"  Part="1"
 F 0 "P13" H 4900 3950 50  0000 C CNN
-F 1 "GP2" V 5000 3750 50  0000 C CNN
+F 1 "GP2_IO" V 5000 3750 50  0000 C CNN
 F 2 "" H 4900 3750 60  0001 C CNN
 F 3 "" H 4900 3750 60  0000 C CNN

Commit message: Updating the schematic's annotations.
Parts:
- renumbered C12 to C801, C13 to C802, P8 to P801, R20 to R801, R21 to R802
Changed lines of the file:
@@
 $EndDescr
 $Comp
-L Conn_01x03 P8
+L Conn_01x03 P801
 U 1 1 55E7C054
 P 4900 3750
-AR Path="/59FB8CCA/55E7C054" Ref="P8"  Part="1"
-AR Path="/59FF5446/55E7C054" Ref="P9"  Part="1"
-AR Path="/59FF5905/55E7C054" Ref="P10"  Part="1"
-AR Path="/59FF590A/55E7C054" Ref="P11"  Part="1"
-AR Path="/59FF5C5D/55E7C054" Ref="P12"  Part="1"
-AR Path="/59FF5C62/55E7C054" Ref="P13"  Part="1"
-F 0 "P13" H 4900 3950 50  0000 C CNN
+AR Path="/59FB8CCA/55E7C054" Ref="P801"  Part="1"
+AR Path="/59FF5446/55E7C054" Ref="P901"  Part="1"
+AR Path="/59FF5905/55E7C054" Ref="P1001"  Part="1"
+AR Path="/59FF590A/55E7C054" Ref="P1101"  Part="1"
+AR Path="/59FF5C5D/55E7C054" Ref="P1201"  Part="1"
+AR Path="/59FF5C62/55E7C054" Ref="P1301"  Part="1"
+F 0 "P1301" H 4900 3950 50  0000 C CNN
 F 1 "GP2_IO" V 5000 3750 50  0000 C CNN
 F 2 "" H 4900 3750 60  0001 C CNN
@@
 $EndComp
 $Comp
-L C C12
+L C C801
 U 1 1 55E7C068
 P 5250 3450
-AR Path="/59FB8CCA/55E7C068" Ref="C12"  Part="1"
-AR Path="/59FF5446/55E7C068" Ref="C14"  Part="1"
-AR Path="/59FF5905/55E7C068" Ref="C16"  Part="1"
-AR Path="/59FF590A/55E7C068" Ref="C18"  Part="1"
-AR Path="/59FF5C5D/55E7C068" Ref="C20"  Part="1"
-AR Path="/59FF5C62/55E7C068" Ref="C22"  Part="1"
-F 0 "C22" H 5275 3550 50  0000 L CNN
+AR Path="/59FB8CCA/55E7C068" Ref="C801"  Part="1"
+AR Path="/59FF5446/55E7C068" Ref="C901"  Part="1"
+AR Path="/59FF5905/55E7C068" Ref="C1001"  Part="1"
+AR Path="/59FF590A/55E7C068" Ref="C1101"  Part="1"
+AR Path="/59FF5C5D/55E7C068" Ref="C1201"  Part="1"
+AR Path="/59FF5C62/55E7C068" Ref="C1301"  Part="1"
+F 0 "C1301" H 5275 3550 50  0000 L CNN
 F 1 "10µF" H 5275 3350 50  0000 L CNN
 F 2 "" H 5288 3300 30  0001 C CNN
@@
 Signal
 $Comp
-L R R20
+L R R801
 U 1 1 55E88E74
 P 5700 3850
-AR Path="/59FB8CCA/55E88E74" Ref="R20"  Part="1"
-AR Path="/59FF5446/55E88E74" Ref="R22"  Part="1"
-AR Path="/59FF5905/55E88E74" Ref="R24"  Part="1"
-AR Path="/59FF590A/55E88E74" Ref="R26"  Part="1"
-AR Path="/59FF5C5D/55E88E74" Ref="R28"  Part="1"
-AR Path="/59FF5C62/55E88E74" Ref="R30"  Part="1"
-F 0 "R30" V 5780 3850 50  0000 C CNN
+AR Path="/59FB8CCA/55E88E74" Ref="R801"  Part="1"
+AR Path="/59FF5446/55E88E74" Ref="R901"  Part="1"
+AR Path="/59FF5905/55E88E74" Ref="R1001"  Part="1"
+AR Path="/59FF590A/55E88E74" Ref="R1101"  Part="1"
+AR Path="/59FF5C5D/55E88E74" Ref="R1201"  Part="1"
+AR Path="/59FF5C62/55E88E74" Ref="R1301"  Part="1"
+F 0 "R1301" V 5780 3850 50  0000 C CNN
 F 1 "10kΩ" V 5700 3850 50  0000 C CNN
 F 2 "" V 5630 3850 30  0001 C CNN
@@
 Connection ~ 5950 3850
 $Comp
-L R R21
+L R R802
 U 1 1 55E88FA1
 P 6200 3850
-AR Path="/59FB8CCA/55E88FA1" Ref="R21"  Part="1"
-AR Path="/59FF5446/55E88FA1" Ref="R23"  Part="1"
-AR Path="/59FF5905/55E88FA1" Ref="R25"  Part="1"
-AR Path="/59FF590A/55E88FA1" Ref="R27"  Part="1"
-AR Path="/59FF5C5D/55E88FA1" Ref="R29"  Part="1"
-AR Path="/59FF5C62/55E88FA1" Ref="R31"  Part="1"
-F 0 "R31" V 6280 3850 50  0000 C CNN
+AR Path="/59FB8CCA/55E88FA1" Ref="R802"  Part="1"
+AR Path="/59FF5446/55E88FA1" Ref="R902"  Part="1"
+AR Path="/59FF5905/55E88FA1" Ref="R1002"  Part="1"
+AR Path="/59FF590A/55E88FA1" Ref="R1102"  Part="1"
+AR Path="/59FF5C5D/55E88FA1" Ref="R1202"  Part="1"
+AR Path="/59FF5C62/55E88FA1" Ref="R1302"  Part="1"
+F 0 "R1302" V 6280 3850 50  0000 C CNN
 F 1 "20kΩ" V 6200 3850 50  0000 C CNN
 F 2 "" V 6130 3850 30  0001 C CNN
@@
 	6350 3450 5400 3450
 $Comp
-L C C13
+L C C802
 U 1 1 5602AA98
 P 5950 3650
-AR Path="/59FB8CCA/5602AA98" Ref="C13"  Part="1"
-AR Path="/59FF5446/5602AA98" Ref="C15"  Part="1"
-AR Path="/59FF5905/5602AA98" Ref="C17"  Part="1"
-AR Path="/59FF590A/5602AA98" Ref="C19"  Part="1"
-AR Path="/59FF5C5D/5602AA98" Ref="C21"  Part="1"
-AR Path="/59FF5C62/5602AA98" Ref="C23"  Part="1"
-F 0 "C23" H 5975 3750 50  0000 L CNN
+AR Path="/59FB8CCA/5602AA98" Ref="C802"  Part="1"
+AR Path="/59FF5446/5602AA98" Ref="C902"  Part="1"
+AR Path="/59FF5905/5602AA98" Ref="C1002"  Part="1"
+AR Path="/59FF590A/5602AA98" Ref="C1102"  Part="1"
+AR Path="/59FF5C5D/5602AA98" Ref="C1202"  Part="1"
+AR Path="/59FF5C62/5602AA98" Ref="C1302"  Part="1"
+F 0 "C1302" H 5975 3750 50  0000 L CNN
 F 1 "100nF" H 5975 3550 50  0000 L CNN
 F 2 "" H 5988 3500 30  0001 C CNN

Commit message: Setting the schematic's footprints.
Parts:
- C801, C802: footprint (none) -> Capacitors_SMD:C_1206_HandSoldering
- P801: footprint (none) -> Connectors_Molex:Molex_KK-6410-03_03x2.54mm_Straight
- R801, R802: footprint (none) -> Resistors_SMD:R_1206_HandSoldering
Changed lines of the file:
@@
 F 0 "P1301" H 4900 3950 50  0000 C CNN
 F 1 "GP2_IO" V 5000 3750 50  0000 C CNN
-F 2 "" H 4900 3750 60  0001 C CNN
+F 2 "Connectors_Molex:Molex_KK-6410-03_03x2.54mm_Straight" H 4900 3750 60  0001 C CNN
 F 3 "" H 4900 3750 60  0000 C CNN
 	1    4900 3750
@@
 F 0 "C1301" H 5275 3550 50  0000 L CNN
 F 1 "10µF" H 5275 3350 50  0000 L CNN
-F 2 "" H 5288 3300 30  0001 C CNN
+F 2 "Capacitors_SMD:C_1206_HandSoldering" H 5288 3300 30  0001 C CNN
 F 3 "" H 5250 3450 60  0000 C CNN
 	1    5250 3450
@@
 F 0 "R1301" V 5780 3850 50  0000 C CNN
 F 1 "10kΩ" V 5700 3850 50  0000 C CNN
-F 2 "" V 5630 3850 30  0001 C CNN
+F 2 "Resistors_SMD:R_1206_HandSoldering" V 5630 3850 30  0001 C CNN
 F 3 "" H 5700 3850 30  0000 C CNN
 	1    5700 3850
@@
 F 0 "R1302" V 6280 3850 50  0000 C CNN
 F 1 "20kΩ" V 6200 3850 50  0000 C CNN
-F 2 "" V 6130 3850 30  0001 C CNN
+F 2 "Resistors_SMD:R_1206_HandSoldering" V 6130 3850 30  0001 C CNN
 F 3 "" H 6200 3850 30  0000 C CNN
 	1    6200 3850
@@
 F 0 "C1302" H 5975 3750 50  0000 L CNN
 F 1 "100nF" H 5975 3550 50  0000 L CNN
-F 2 "" H 5988 3500 30  0001 C CNN
+F 2 "Capacitors_SMD:C_1206_HandSoldering" H 5988 3500 30  0001 C CNN
 F 3 "" H 5950 3650 60  0000 C CNN
 	1    5950 3650
