File: Power.sch (KiCad schematic (older format))
At the start: 3 parts, among them P5 Bat5V, P6 Bat15V

Commit message: Adding Hermes 2 schematic files.
Parts:
- removed P5: Bat5V, Footprints:Conn_01x02, symbol CONN_01X02
- added C1: 10µF, symbol C
- added C2: 220nF, symbol C
- added C3: 1µF, symbol C
- added C4: 100nF, symbol C
- added D4: LED_15V, symbol LED
- added D5: LED_5V, symbol LED
- added P1: Power IO, symbol Conn_01x03
- added R4: 6kΩ, symbol R
- added R5: 1.4kΩ, symbol R
- added U2: LM7805, symbol LM7805_TO220
- F1: footprint Footprints:Fuse -> (none); symbol FUSE -> Fuse
- P2: renamed from P6; value Bat15V -> Power IO; footprint Footprints:Power_Conn_01x02 -> (none); symbol CONN_01X02 -> Conn_01x03
Connections:
- wire segments 6 -> 28

Commit message: Moving the 5V regulator to the non-emergency-stop-guarded +15V and adding a fuse for it.
Parts:
- added F1: FUSE 30A, symbol Fuse
- F2: renamed from F1; value FUSE -> FUSE 1A
Connections:
- wire segments 28 -> 29
Other:
- moved on the sheet: C1, C2, C3, C4, D4, D5, R4, R5

Commit message: Changing some value fields on the schematics for a better grouped_csv BOM generation.
Parts:
- P1, P2: value Power IO -> Power_IO
Changed lines of the file:
@@
 P 4150 3500
 F 0 "P2" H 4150 3700 50  0000 C CNN
-F 1 "Power IO" V 4250 3500 50  0000 C CNN
+F 1 "Power_IO" V 4250 3500 50  0000 C CNN
 F 2 "" H 4150 3500 60  0001 C CNN
 F 3 "" H 4150 3500 60  0000 C CNN
@@
 P 4150 2950
 F 0 "P1" H 4150 3150 50  0000 C CNN
-F 1 "Power IO" V 4250 2950 50  0000 C CNN
+F 1 "Power_IO" V 4250 2950 50  0000 C CNN
 F 2 "" H 4150 2950 60  0001 C CNN
 F 3 "" H 4150 2950 60  0000 C CNN

Commit message: Changing the LM7805 for a OKI78SR5/1.5W36C since it would heat way too much with a +15V input.
Parts:
- U2: value LM7805 -> OKI78SR5/1.5W36C
Changed lines of the file:
@@
 P 6250 3400
 F 0 "U2" H 6100 3525 50  0000 C CNN
-F 1 "LM7805" H 6250 3525 50  0000 L CNN
+F 1 "OKI78SR5/1.5W36C" H 5850 3600 50  0000 L CNN
 F 2 "" H 6250 3625 50  0001 C CIN
 F 3 "" H 6250 3350 50  0001 C CNN

Commit message: Replacing the 5V regulator's input 220nF capacitor with two 100nF capacitors.
Parts:
- added C?: 100nF, symbol C
- C2: value 220nF -> 100nF
Connections:
- wire segments 29 -> 31
Other:
- moved on the sheet: C3, C4, D5, R5
Changed lines of the file:
@@
 	-1   0    0    -1
 $EndComp
-Text HLabel 6650 3300 1    60   Output ~ 0
+Text HLabel 6900 3300 1    60   Output ~ 0
 +5V
 Text HLabel 4650 4600 3    60   Output ~ 0
@@
 P 5850 3650
 F 0 "C2" H 5875 3750 50  0000 L CNN
-F 1 "220nF" H 5875 3550 50  0000 L CNN
+F 1 "100nF" H 5875 3550 50  0000 L CNN
 F 2 "" H 5888 3500 50  0001 C CNN
 F 3 "" H 5850 3650 50  0001 C CNN
@@
 L C C4
 U 1 1 59FBAF9E
-P 6900 3650
-F 0 "C4" H 6925 3750 50  0000 L CNN
-F 1 "100nF" H 6925 3550 50  0000 L CNN
-F 2 "" H 6938 3500 50  0001 C CNN
-F 3 "" H 6900 3650 50  0001 C CNN
-	1    6900 3650
+P 7150 3650
+F 0 "C4" H 7175 3750 50  0000 L CNN
+F 1 "100nF" H 7175 3550 50  0000 L CNN
+F 2 "" H 7188 3500 50  0001 C CNN
+F 3 "" H 7150 3650 50  0001 C CNN
+	1    7150 3650
 	1    0    0    -1
 $EndComp
@@
 L C C3
 U 1 1 59FF29CD
-P 6650 3650
-F 0 "C3" H 6675 3750 50  0000 L CNN
-F 1 "1µF" H 6675 3550 50  0000 L CNN
-F 2 "" H 6688 3500 50  0001 C CNN
-F 3 "" H 6650 3650 50  0001 C CNN
-	1    6650 3650
+P 6900 3650
+F 0 "C3" H 6925 3750 50  0000 L CNN
+F 1 "1µF" H 6925 3550 50  0000 L CNN
+F 2 "" H 6938 3500 50  0001 C CNN
+F 3 "" H 6900 3650 50  0001 C CNN
+	1    6900 3650
 	1    0    0    -1
 $EndComp
@@
 L LM7805_TO220 U2
 U 1 1 59FBAA64
-P 6250 3400
-F 0 "U2" H 6100 3525 50  0000 C CNN
-F 1 "OKI78SR5/1.5W36C" H 5850 3600 50  0000 L CNN
-F 2 "" H 6250 3625 50  0001 C CIN
-F 3 "" H 6250 3350 50  0001 C CNN
-	1    6250 3400
+P 6500 3400
+F 0 "U2" H 6350 3525 50  0000 C CNN
+F 1 "OKI78SR5/1.5W36C" H 6100 3600 50  0000 L CNN
+F 2 "" H 6500 3625 50  0001 C CIN
+F 3 "" H 6500 3350 50  0001 C CNN
+	1    6500 3400
 	1    0    0    -1
 $EndComp
@@
 L LED D5
 U 1 1 59FF3CBB
-P 7250 4050
-F 0 "D5" H 7250 4150 50  0000 C CNN
-F 1 "LED_5V" H 7250 3950 50  0000 C CNN
-F 2 "" H 7250 4050 50  0001 C CNN
-F 3 "" H 7250 4050 50  0001 C CNN
-	1    7250 4050
+P 7500 4050
+F 0 "D5" H 7500 4150 50  0000 C CNN
+F 1 "LED_5V" H 7500 3950 50  0000 C CNN
+F 2 "" H 7500 4050 50  0001 C CNN
+F 3 "" H 7500 4050 50  0001 C CNN
+	1    7500 4050
 	0    -1   -1   0
 $EndComp
@@
 L R R5
 U 1 1 59FF3CC1
-P 7250 3650
-F 0 "R5" V 7330 3650 50  0000 C CNN
-F 1 "1.4kΩ" V 7250 3650 50  0000 C CNN
-F 2 "" V 7180 3650 50  0001 C CNN
-F 3 "" H 7250 3650 50  0001 C CNN
-	1    7250 3650
+P 7500 3650
+F 0 "R5" V 7580 3650 50  0000 C CNN
+F 1 "1.4kΩ" V 7500 3650 50  0000 C CNN
+F 2 "" V 7430 3650 50  0001 C CNN
+F 3 "" H 7500 3650 50  0001 C CNN
+	1    7500 3650
 	1    0    0    -1
 $EndComp
@@
 $EndComp
 Wire Wire Line
-	5850 3400 5850 3500
-Wire Wire Line
 	5050 4000 5050 4100
 Wire Wire Line
-	7250 3800 7250 3900
-Wire Wire Line
-	6550 3400 7250 3400
-Wire Wire Line
-	6650 3300 6650 3500
-Wire Wire Line
-	6900 3400 6900 3500
-Connection ~ 6650 3400
-Wire Wire Line
-	7250 3400 7250 3500
+	7500 3800 7500 3900
+Wire Wire Line
+	6800 3400 7500 3400
+Wire Wire Line
+	6900 3300 6900 3500
+Wire Wire Line
+	7150 3400 7150 3500
 Connection ~ 6900 3400
+Wire Wire Line
+	7500 3400 7500 3500
+Connection ~ 7150 3400
 Wire Wire Line
 	5600 3500 5600 3400
 Connection ~ 5600 3400
-Wire Wire Line
-	5500 3400 5950 3400
-Connection ~ 5850 3400
 Wire Wire Line
 	4350 2950 4550 2950
@@
 Connection ~ 5050 3600
 Wire Wire Line
-	4550 4500 7250 4500
-Wire Wire Line
 	4650 4500 4650 4600
 Connection ~ 4550 3500
@@
 Connection ~ 5600 4500
 Wire Wire Line
-	6250 4500 6250 3700
+	6500 4500 6500 3700
 Connection ~ 5850 4500
 Wire Wire Line
-	6650 4500 6650 3800
-Connection ~ 6250 4500
-Wire Wire Line
 	6900 4500 6900 3800
-Connection ~ 6650 4500
-Wire Wire Line
-	7250 4500 7250 4200
+Connection ~ 6500 4500
+Wire Wire Line
+	7150 4500 7150 3800
 Connection ~ 6900 4500
+Wire Wire Line
+	7500 4500 7500 4200
+Connection ~ 7150 4500
+Wire Wire Line
+	5850 3400 5850 3500
+Connection ~ 5850 3400
+Wire Wire Line
+	4550 4500 7500 4500
+$Comp
+L C C?
+U 1 1 5A3EA598
+P 6100 3650
+F 0 "C?" H 6125 3750 50  0000 L CNN
+F 1 "100nF" H 6125 3550 50  0000 L CNN
+F 2 "" H 6138 3500 50  0001 C CNN
+F 3 "" H 6100 3650 50  0001 C CNN
+	1    6100 3650
+	1    0    0    -1
+$EndComp
+Wire Wire Line
+	5500 3400 6200 3400
+Wire Wire Line
+	6100 3400 6100 3500
+Connection ~ 6100 3400
+Wire Wire Line
+	6100 3800 6100 4500
+Connection ~ 6100 4500
 $EndSCHEMATC

Commit message: Updating the schematic's annotations.
Parts:
- gave numbers to parts that had none: 1
- renumbered C1 to C201, C2 to C202, C3 to C204, C4 to C205, D4 to D201, D5 to D202, F1 to F201, F2 to F202, P1 to P201, P2 to P202, R4 to R201, R5 to R202, U2 to U201
Changed lines of the file:
@@
 $EndDescr
 $Comp
-L Conn_01x03 P2
+L Conn_01x03 P202
 U 1 1 55E7E313
 P 4150 3500
-F 0 "P2" H 4150 3700 50  0000 C CNN
+F 0 "P202" H 4150 3700 50  0000 C CNN
 F 1 "Power_IO" V 4250 3500 50  0000 C CNN
 F 2 "" H 4150 3500 60  0001 C CNN
@@
 +15V
 $Comp
-L Fuse F2
+L Fuse F202
 U 1 1 560397C6
 P 5350 3400
-F 0 "F2" V 5450 3400 50  0000 C CNN
+F 0 "F202" V 5450 3400 50  0000 C CNN
 F 1 "FUSE 1A" V 5250 3400 50  0000 C CNN
 F 2 "" H 5350 3400 60  0001 C CNN
@@
 $EndComp
 $Comp
-L C C2
+L C C202
 U 1 1 59FBAE48
 P 5850 3650
-F 0 "C2" H 5875 3750 50  0000 L CNN
+F 0 "C202" H 5875 3750 50  0000 L CNN
 F 1 "100nF" H 5875 3550 50  0000 L CNN
 F 2 "" H 5888 3500 50  0001 C CNN
@@
 $EndComp
 $Comp
-L C C4
+L C C205
 U 1 1 59FBAF9E
 P 7150 3650
-F 0 "C4" H 7175 3750 50  0000 L CNN
+F 0 "C205" H 7175 3750 50  0000 L CNN
 F 1 "100nF" H 7175 3550 50  0000 L CNN
 F 2 "" H 7188 3500 50  0001 C CNN
@@
 $EndComp
 $Comp
-L C C1
+L C C201
 U 1 1 59FF296D
 P 5600 3650
-F 0 "C1" H 5625 3750 50  0000 L CNN
+F 0 "C201" H 5625 3750 50  0000 L CNN
 F 1 "10µF" H 5625 3550 50  0000 L CNN
 F 2 "" H 5638 3500 50  0001 C CNN
@@
 $EndComp
 $Comp
-L C C3
+L C C204
 U 1 1 59FF29CD
 P 6900 3650
-F 0 "C3" H 6925 3750 50  0000 L CNN
+F 0 "C204" H 6925 3750 50  0000 L CNN
 F 1 "1µF" H 6925 3550 50  0000 L CNN
 F 2 "" H 6938 3500 50  0001 C CNN
@@
 $EndComp
 $Comp
-L LED D4
+L LED D201
 U 1 1 59FF376D
 P 5050 4250
-F 0 "D4" H 5050 4350 50  0000 C CNN
+F 0 "D201" H 5050 4350 50  0000 C CNN
 F 1 "LED_15V" H 5050 4150 50  0000 C CNN
 F 2 "" H 5050 4250 50  0001 C CNN
@@
 $EndComp
 $Comp
-L LM7805_TO220 U2
+L LM7805_TO220 U201
 U 1 1 59FBAA64
 P 6500 3400
-F 0 "U2" H 6350 3525 50  0000 C CNN
+F 0 "U201" H 6350 3525 50  0000 C CNN
 F 1 "OKI78SR5/1.5W36C" H 6100 3600 50  0000 L CNN
 F 2 "" H 6500 3625 50  0001 C CIN
@@
 $EndComp
 $Comp
-L R R4
+L R R201
 U 1 1 59FF39F1
 P 5050 3850
-F 0 "R4" V 5130 3850 50  0000 C CNN
+F 0 "R201" V 5130 3850 50  0000 C CNN
 F 1 "6kΩ" V 5050 3850 50  0000 C CNN
 F 2 "" V 4980 3850 50  0001 C CNN
@@
 $EndComp
 $Comp
-L LED D5
+L LED D202
 U 1 1 59FF3CBB
 P 7500 4050
-F 0 "D5" H 7500 4150 50  0000 C CNN
+F 0 "D202" H 7500 4150 50  0000 C CNN
 F 1 "LED_5V" H 7500 3950 50  0000 C CNN
 F 2 "" H 7500 4050 50  0001 C CNN
@@
 $EndComp
 $Comp
-L R R5
+L R R202
 U 1 1 59FF3CC1
 P 7500 3650
-F 0 "R5" V 7580 3650 50  0000 C CNN
+F 0 "R202" V 7580 3650 50  0000 C CNN
 F 1 "1.4kΩ" V 7500 3650 50  0000 C CNN
 F 2 "" V 7430 3650 50  0001 C CNN
@@
 $EndComp
 $Comp
-L Conn_01x03 P1
+L Conn_01x03 P201
 U 1 1 5A049EFB
 P 4150 2950
-F 0 "P1" H 4150 3150 50  0000 C CNN
+F 0 "P201" H 4150 3150 50  0000 C CNN
 F 1 "Power_IO" V 4250 2950 50  0000 C CNN
 F 2 "" H 4150 2950 60  0001 C CNN
@@
 $EndComp
 $Comp
-L Fuse F1
+L Fuse F201
 U 1 1 5A10A9EC
 P 4800 3600
-F 0 "F1" V 4900 3600 50  0000 C CNN
+F 0 "F201" V 4900 3600 50  0000 C CNN
 F 1 "FUSE 30A" V 4700 3600 50  0000 C CNN
 F 2 "" H 4800 3600 60  0001 C CNN
@@
 	4550 4500 7500 4500
 $Comp
-L C C?
+L C C203
 U 1 1 5A3EA598
 P 6100 3650
-F 0 "C?" H 6125 3750 50  0000 L CNN
+F 0 "C203" H 6125 3750 50  0000 L CNN
 F 1 "100nF" H 6125 3550 50  0000 L CNN
 F 2 "" H 6138 3500 50  0001 C CNN

Commit message: Setting the schematic's footprints.
Parts:
- C201, C202, C203, C204, C205: footprint (none) -> Capacitors_SMD:C_1206_HandSoldering
- D201, D202: footprint (none) -> LEDs:LED_1206_HandSoldering
- F201: footprint (none) -> xenocad.fuses:Fuse_Eaton-ABC_20A+_Axial
- F202: footprint (none) -> xenocad.fuses:Fuseholder_Littlefuse-646
- P201, P202: footprint (none) -> xenocad.connectors:Hirose_DF22-03P-7.92DS_03x7.92mm_Angled
- R201, R202: footprint (none) -> Resistors_SMD:R_1206_HandSoldering
- U201: footprint (none) -> xenocad.regul:OKI-78SR-Vertical
Changed lines of the file:
@@
 F 0 "P202" H 4150 3700 50  0000 C CNN
 F 1 "Power_IO" V 4250 3500 50  0000 C CNN
-F 2 "" H 4150 3500 60  0001 C CNN
+F 2 "xenocad.connectors:Hirose_DF22-03P-7.92DS_03x7.92mm_Angled" H 4150 3500 60  0001 C CNN
 F 3 "" H 4150 3500 60  0000 C CNN
 	1    4150 3500
@@
 F 0 "F202" V 5450 3400 50  0000 C CNN
 F 1 "FUSE 1A" V 5250 3400 50  0000 C CNN
-F 2 "" H 5350 3400 60  0001 C CNN
+F 2 "xenocad.fuses:Fuseholder_Littlefuse-646" H 5350 3400 60  0001 C CNN
 F 3 "" H 5350 3400 60  0000 C CNN
 	1    5350 3400
@@
 F 0 "C202" H 5875 3750 50  0000 L CNN
 F 1 "100nF" H 5875 3550 50  0000 L CNN
-F 2 "" H 5888 3500 50  0001 C CNN
+F 2 "Capacitors_SMD:C_1206_HandSoldering" H 5888 3500 50  0001 C CNN
 F 3 "" H 5850 3650 50  0001 C CNN
 	1    5850 3650
@@
 F 0 "C205" H 7175 3750 50  0000 L CNN
 F 1 "100nF" H 7175 3550 50  0000 L CNN
-F 2 "" H 7188 3500 50  0001 C CNN
+F 2 "Capacitors_SMD:C_1206_HandSoldering" H 7188 3500 50  0001 C CNN
 F 3 "" H 7150 3650 50  0001 C CNN
 	1    7150 3650
@@
 F 0 "C201" H 5625 3750 50  0000 L CNN
 F 1 "10µF" H 5625 3550 50  0000 L CNN
-F 2 "" H 5638 3500 50  0001 C CNN
+F 2 "Capacitors_SMD:C_1206_HandSoldering" H 5638 3500 50  0001 C CNN
 F 3 "" H 5600 3650 50  0001 C CNN
 	1    5600 3650
@@
 F 0 "C204" H 6925 3750 50  0000 L CNN
 F 1 "1µF" H 6925 3550 50  0000 L CNN
-F 2 "" H 6938 3500 50  0001 C CNN
+F 2 "Capacitors_SMD:C_1206_HandSoldering" H 6938 3500 50  0001 C CNN
 F 3 "" H 6900 3650 50  0001 C CNN
 	1    6900 3650
@@
 F 0 "D201" H 5050 4350 50  0000 C CNN
 F 1 "LED_15V" H 5050 4150 50  0000 C CNN
-F 2 "" H 5050 4250 50  0001 C CNN
+F 2 "LEDs:LED_1206_HandSoldering" H 5050 4250 50  0001 C CNN
 F 3 "" H 5050 4250 50  0001 C CNN
 	1    5050 4250
@@
 F 0 "U201" H 6350 3525 50  0000 C CNN
 F 1 "OKI78SR5/1.5W36C" H 6100 3600 50  0000 L CNN
-F 2 "" H 6500 3625 50  0001 C CIN
+F 2 "xenocad.regul:OKI-78SR-Vertical" H 6500 3625 50  0001 C CIN
 F 3 "" H 6500 3350 50  0001 C CNN
 	1    6500 3400
@@
 F 0 "R201" V 5130 3850 50  0000 C CNN
 F 1 "6kΩ" V 5050 3850 50  0000 C CNN
-F 2 "" V 4980 3850 50  0001 C CNN
+F 2 "Resistors_SMD:R_1206_HandSoldering" V 4980 3850 50  0001 C CNN
 F 3 "" H 5050 3850 50  0001 C CNN
 	1    5050 3850
@@
 F 0 "D202" H 7500 4150 50  0000 C CNN
 F 1 "LED_5V" H 7500 3950 50  0000 C CNN
-F 2 "" H 7500 4050 50  0001 C CNN
+F 2 "LEDs:LED_1206_HandSoldering" H 7500 4050 50  0001 C CNN
 F 3 "" H 7500 4050 50  0001 C CNN
 	1    7500 4050
@@
 F 0 "R202" V 7580 3650 50  0000 C CNN
 F 1 "1.4kΩ" V 7500 3650 50  0000 C CNN
-F 2 "" V 7430 3650 50  0001 C CNN
+F 2 "Resistors_SMD:R_1206_HandSoldering" V 7430 3650 50  0001 C CNN
 F 3 "" H 7500 3650 50  0001 C CNN
 	1    7500 3650
@@
 F 0 "P201" H 4150 3150 50  0000 C CNN
 F 1 "Power_IO" V 4250 2950 50  0000 C CNN
-F 2 "" H 4150 2950 60  0001 C CNN
+F 2 "xenocad.connectors:Hirose_DF22-03P-7.92DS_03x7.92mm_Angled" H 4150 2950 60  0001 C CNN
 F 3 "" H 4150 2950 60  0000 C CNN
 	1    4150 2950
@@
 F 0 "F201" V 4900 3600 50  0000 C CNN
 F 1 "FUSE 30A" V 4700 3600 50  0000 C CNN
-F 2 "" H 4800 3600 60  0001 C CNN
+F 2 "xenocad.fuses:Fuse_Eaton-ABC_20A+_Axial" H 4800 3600 60  0001 C CNN
 F 3 "" H 4800 3600 60  0000 C CNN
 	1    4800 3600
@@
 F 0 "C203" H 6125 3750 50  0000 L CNN
 F 1 "100nF" H 6125 3550 50  0000 L CNN
-F 2 "" H 6138 3500 50  0001 C CNN
+F 2 "Capacitors_SMD:C_1206_HandSoldering" H 6138 3500 50  0001 C CNN
 F 3 "" H 6100 3650 50  0001 C CNN
 	1    6100 3650
